File: schematics/Laser_Targeting_System/laser_pcb.brd (EAGLE design)
At the start: 50.8 x 56.5 mm, 28 parts, among them IC2 ATMEGA328-PU, J1 CON-SOCJ-2155, J2 292304-1, K1 G5LE, Q2 PN2222

Commit message: updated schematic
Connections:
- removed net N$1: C5.2, IC2.1, RESET.1, TX/RX/RESET.1
- net +5V: now also R1-RESET.2; no longer R1-RESET.1
- net GND: now also RESET.3
- net N$4: now also C5.2, IC2.1, R1-RESET.1, RESET.1, TX/RX/RESET.1; no longer R1-RESET.2, RESET.3
Routing:
- net N$1: track 71.9 -> 0.00 mm, vias 4 -> 0
- net N$4: track 91.4 -> 66.0 mm, vias 1 -> 5
- net GND: track 237.8 -> 246.7 mm
- net +5V: track 141.6 -> 149.2 mm, vias 7 -> 8

Commit message: updated schematic
Routing:
- net GND: track 246.7 -> 0.00 mm, vias 4 -> 0
